File: Hardware/matrix.kicad_sch (KiCad schematic)
At the start: 258 parts, among them SW1 SW_Push, SW10 SW_Push, SW100 SW_Push, SW101 SW_Push, SW102 SW_Push, SW103 SW_Push, SW104 SW_Push, SW105 SW_Push, SW106 SW_Push, SW107 SW_Push, SW108 SW_Push, SW109 SW_Push, SW11 SW_Push, SW110 SW_Push, SW111 SW_Push, SW112 SW_Push, SW113 SW_Push, SW114 SW_Push, SW115 SW_Push, SW116 SW_Push, SW117 SW_Push, SW118 SW_Push, SW119 SW_Push, SW12 SW_Push, SW120 SW_Push, SW121 SW_Push, SW122 SW_Push, SW123 SW_Push, SW124 SW_Push, SW125 SW_Push, SW126 SW_Push, SW127 SW_Push, SW128 SW_Push, SW129 SW_Push, SW13 SW_Push, SW14 SW_Push, SW15 SW_Push, SW16 SW_Push, SW17 SW_Push, SW18 SW_Push, SW19 SW_Push, SW2 SW_Push, SW20 SW_Push, SW21 SW_Push, SW22 SW_Push, SW23 SW_Push, SW24 SW_Push, SW25 SW_Push, SW26 SW_Push, SW27 SW_Push, SW28 SW_Push, SW29 SW_Push, SW3 SW_Push, SW30 SW_Push, SW31 SW_Push, SW32 SW_Push, SW33 SW_Push, SW34 SW_Push, SW35 SW_Push, SW36 SW_Push, SW37 SW_Push, SW38 SW_Push, SW39 SW_Push, SW4 SW_Push, SW40 SW_Push, SW41 SW_Push, SW42 SW_Push, SW43 SW_Push, SW44 SW_Push, SW45 SW_Push, SW46 SW_Push, SW47 SW_Push, SW48 SW_Push, SW49 SW_Push, SW5 SW_Push, SW50 SW_Push, SW51 SW_Push, SW52 SW_Push, SW53 SW_Push, SW54 SW_Push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

Commit message: Final design for v2.0
Parts:
- D2, SW2: now not fitted
Changed lines of the file:
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@@
   )
   (symbol (lib_id "Device:D") (at 46.99 38.735 90) (unit 1)
-    (in_bom yes) (on_board yes) (dnp no) (fields_autoplaced)
+    (in_bom yes) (on_board no) (dnp yes) (fields_autoplaced)
     (property "Reference" "D2" (at 49.022 37.8265 90)
       (effects (font (size 1.27 1.27)) (justify right))
@@
   )
   (symbol (lib_id "Switch:SW_Push") (at 52.07 34.925 0) (unit 1)
-    (in_bom yes) (on_board yes) (dnp no) (fields_autoplaced)
+    (in_bom yes) (on_board no) (dnp yes) (fields_autoplaced)
     (property "Reference" "SW2" (at 52.07 28.0375 0)
       (effects (font (size 1.27 1.27)))
